File: perma-proto-board-v1/perma-proto-board.kicad_sch (KiCad schematic)
At the start: 46 parts, among them J1 SPI_01, J10 I2C_04, J11 I2C_05, J12 I2C_06, J13 A_1, J14 A_2, J15 A_3, J16 A_4, J17 A_5, J18 B_1, J19 B_2, J2 SPI_02, J20 B_3, J21 B_4, J22 B_5, J23 C_1, J24 C_2, J25 C_3, J26 C_4, J27 C_5, J28 Power01, J29 Power02, J3 SPI_03, J30 Power03, J31 Power04, J32 Rail01, J33 Rail02, J34 Rail03, J35 Rail04, J36 Rail05, J37 Rail06, J38 Rail07, J39 Rail08, J4 SPI_04, J40 USB_C_Receptacle, J41 SPI_CS_01, J42 SPI_CS_02, J43 SPI_CS_03, J44 SPI_CS_04, J45 SPI_CS_05, J46 SPI_CS_06, J5 SPI_05, J6 SPI_06, J7 I2C_01, J8 I2C_02, J9 I2C_03

Commit message: v1.1
Parts:
- J13, J14, J15, J16, J17, J18, J19, J20, J21, J22, J23, J24, J25, J26, J27, J32, J33, J34, J35, J36, J37, J38, J39: footprint Connector_PinHeader_2.54mm:PinHeader_1x40_P2.54mm_Vertical -> perma-proto-board-v1:PinHeader_1x40_P2.54mm_Vertical_NO_Silk

Commit message: silk screen fix
Parts:
- J32, J33, J34, J35, J36, J37, J38, J39: footprint perma-proto-board-v1:PinHeader_1x40_P2.54mm_Vertical_NO_Silk -> Connector_PinHeader_2.54mm:PinHeader_1x40_P2.54mm_Vertical
Changed lines of the file:
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@@
     (property "Reference" "J34" (id 0) (at 123.825 159.385 90))
     (property "Value" "Rail03" (id 1) (at 125.73 162.56 90))
-    (property "Footprint" "perma-proto-board-v1:PinHeader_1x40_P2.54mm_Vertical_NO_Silk" (id 2) (at 72.39 158.115 0)
+    (property "Footprint" "Connector_PinHeader_2.54mm:PinHeader_1x40_P2.54mm_Vertical" (id 2) (at 72.39 158.115 0)
       (effects (font (size 1.27 1.27)) hide)
     )
@@
     (property "Reference" "J35" (id 0) (at 123.825 173.99 90))
     (property "Value" "Rail04" (id 1) (at 125.73 177.165 90))
-    (property "Footprint" "perma-proto-board-v1:PinHeader_1x40_P2.54mm_Vertical_NO_Silk" (id 2) (at 72.39 172.72 0)
+    (property "Footprint" "Connector_PinHeader_2.54mm:PinHeader_1x40_P2.54mm_Vertical" (id 2) (at 72.39 172.72 0)
       (effects (font (size 1.27 1.27)) hide)
     )
@@
     (property "Reference" "J38" (id 0) (at 123.825 216.535 90))
     (property "Value" "Rail07" (id 1) (at 125.73 219.71 90))
-    (property "Footprint" "perma-proto-board-v1:PinHeader_1x40_P2.54mm_Vertical_NO_Silk" (id 2) (at 72.39 215.265 0)
+    (property "Footprint" "Connector_PinHeader_2.54mm:PinHeader_1x40_P2.54mm_Vertical" (id 2) (at 72.39 215.265 0)
       (effects (font (size 1.27 1.27)) hide)
     )
@@
     (property "Reference" "J37" (id 0) (at 123.825 201.93 90))
     (property "Value" "Rail06" (id 1) (at 125.73 205.105 90))
-    (property "Footprint" "perma-proto-board-v1:PinHeader_1x40_P2.54mm_Vertical_NO_Silk" (id 2) (at 72.39 200.66 0)
+    (property "Footprint" "Connector_PinHeader_2.54mm:PinHeader_1x40_P2.54mm_Vertical" (id 2) (at 72.39 200.66 0)
       (effects (font (size 1.27 1.27)) hide)
     )
@@
     (property "Reference" "J36" (id 0) (at 123.825 187.325 90))
     (property "Value" "Rail05" (id 1) (at 125.73 190.5 90))
-    (property "Footprint" "perma-proto-board-v1:PinHeader_1x40_P2.54mm_Vertical_NO_Silk" (id 2) (at 72.39 186.055 0)
+    (property "Footprint" "Connector_PinHeader_2.54mm:PinHeader_1x40_P2.54mm_Vertical" (id 2) (at 72.39 186.055 0)
       (effects (font (size 1.27 1.27)) hide)
     )
@@
     (property "Reference" "J32" (id 0) (at 123.825 131.445 90))
     (property "Value" "Rail01" (id 1) (at 125.73 134.62 90))
-    (property "Footprint" "perma-proto-board-v1:PinHeader_1x40_P2.54mm_Vertical_NO_Silk" (id 2) (at 72.39 130.175 0)
+    (property "Footprint" "Connector_PinHeader_2.54mm:PinHeader_1x40_P2.54mm_Vertical" (id 2) (at 72.39 130.175 0)
       (effects (font (size 1.27 1.27)) hide)
     )
@@
     (property "Reference" "J33" (id 0) (at 123.825 145.415 90))
     (property "Value" "Rail02" (id 1) (at 125.73 148.59 90))
-    (property "Footprint" "perma-proto-board-v1:PinHeader_1x40_P2.54mm_Vertical_NO_Silk" (id 2) (at 72.39 144.145 0)
+    (property "Footprint" "Connector_PinHeader_2.54mm:PinHeader_1x40_P2.54mm_Vertical" (id 2) (at 72.39 144.145 0)
       (effects (font (size 1.27 1.27)) hide)
     )
@@
     (property "Reference" "J39" (id 0) (at 123.825 233.68 90))
     (property "Value" "Rail08" (id 1) (at 125.73 236.855 90))
-    (property "Footprint" "perma-proto-board-v1:PinHeader_1x40_P2.54mm_Vertical_NO_Silk" (id 2) (at 72.39 232.41 0)
+    (property "Footprint" "Connector_PinHeader_2.54mm:PinHeader_1x40_P2.54mm_Vertical" (id 2) (at 72.39 232.41 0)
       (effects (font (size 1.27 1.27)) hide)
     )
@@
     )
     (path "/645e71f6-577c-4953-ad6e-62f2240c420b"
-      (reference "J32") (unit 1) (value "Rail01") (footprint "perma-proto-board-v1:PinHeader_1x40_P2.54mm_Vertical_NO_Silk")
+      (reference "J32") (unit 1) (value "Rail01") (footprint "Connector_PinHeader_2.54mm:PinHeader_1x40_P2.54mm_Vertical")
     )
     (path "/a6511fbb-8ce6-4e67-bad0-a0845e467e4e"
-      (reference "J33") (unit 1) (value "Rail02") (footprint "perma-proto-board-v1:PinHeader_1x40_P2.54mm_Vertical_NO_Silk")
+      (reference "J33") (unit 1) (value "Rail02") (footprint "Connector_PinHeader_2.54mm:PinHeader_1x40_P2.54mm_Vertical")
     )
     (path "/1623f3b2-2fa6-4882-90bc-9b99a932a022"
-      (reference "J34") (unit 1) (value "Rail03") (footprint "perma-proto-board-v1:PinHeader_1x40_P2.54mm_Vertical_NO_Silk")
+      (reference "J34") (unit 1) (value "Rail03") (footprint "Connector_PinHeader_2.54mm:PinHeader_1x40_P2.54mm_Vertical")
     )
     (path "/18c60b7d-4c72-4218-9c2a-60573689618b"
-      (reference "J35") (unit 1) (value "Rail04") (footprint "perma-proto-board-v1:PinHeader_1x40_P2.54mm_Vertical_NO_Silk")
+      (reference "J35") (unit 1) (value "Rail04") (footprint "Connector_PinHeader_2.54mm:PinHeader_1x40_P2.54mm_Vertical")
     )
     (path "/45db4970-97e0-45e5-84b0-48b54ade450f"
-      (reference "J36") (unit 1) (value "Rail05") (footprint "perma-proto-board-v1:PinHeader_1x40_P2.54mm_Vertical_NO_Silk")
+      (reference "J36") (unit 1) (value "Rail05") (footprint "Connector_PinHeader_2.54mm:PinHeader_1x40_P2.54mm_Vertical")
     )
     (path "/3c3978c4-7a61-410b-897b-97600062cd09"
-      (reference "J37") (unit 1) (value "Rail06") (footprint "perma-proto-board-v1:PinHeader_1x40_P2.54mm_Vertical_NO_Silk")
+      (reference "J37") (unit 1) (value "Rail06") (footprint "Connector_PinHeader_2.54mm:PinHeader_1x40_P2.54mm_Vertical")
     )
     (path "/30ba56e2-59eb-4dd6-919f-84dd9ed482cc"
-      (reference "J38") (unit 1) (value "Rail07") (footprint "perma-proto-board-v1:PinHeader_1x40_P2.54mm_Vertical_NO_Silk")
+      (reference "J38") (unit 1) (value "Rail07") (footprint "Connector_PinHeader_2.54mm:PinHeader_1x40_P2.54mm_Vertical")
     )
     (path "/d8bb74ea-b054-4a6b-ab5f-68f403fc58cf"
-      (reference "J39") (unit 1) (value "Rail08") (footprint "perma-proto-board-v1:PinHeader_1x40_P2.54mm_Vertical_NO_Silk")
+      (reference "J39") (unit 1) (value "Rail08") (footprint "Connector_PinHeader_2.54mm:PinHeader_1x40_P2.54mm_Vertical")
     )
     (path "/74da7767-fbd4-4d7f-9ec8-5055445d8f7b"
